Commit message: Change name velodyne_link to velodyne

File: orange_description/xacro/sensors/velodyne.xacro (robot description, xacro)
@@ -6,7 +6,7 @@
       <axis xyz="0 1 0"/>
       <parent link="${parent}"/>
-      <child link="${name}_link"/>
+      <child link="${name}"/>
     </joint>
-    <link name="${name}_link">
+    <link name="${name}">
       <visual>
         <origin xyz="0 0 0" rpy="0 0 0"/>
@@ -27,5 +27,5 @@
       </inertial>
     </link>
-    <gazebo reference="${name}_link">
+    <gazebo reference="${name}">
       <sensor type="ray" name="head_velodyne_sensor">
         <pose>0 0 0 0 0 0</pose>
@@ -62,5 +62,5 @@
             <remapping>~/out:=velodyne_points</remapping>
           </ros>
-          <frame_name>${name}_link</frame_name>
+          <frame_name>${name}</frame_name>
           <min_range>0.9</min_range>
           <max_range>100</max_range>

Commit message: Change velodyne spec in xacro

File: orange_description/xacro/sensors/velodyne.xacro (robot description, xacro)
@@ -1,4 +1,5 @@
 <?xml version="1.0"?>
 <robot xmlns:xacro="http://ros.org/wiki/xacro" xmlns:controller="http://playerstage.sourceforge.net/gazebo/xmlschema/#controller" xmlns:interface="http://playerstage.sourceforge.net/gazebo/xmlschema/#interface" name="sensor_velodyne">
+  <xacro:property name="PI" value="3.1415926535897931"/>
   <xacro:macro name="sensor_velodyne" params="name parent *origin min_angle max_angle samples">
     <joint name="${name}_joint" type="fixed">
@@ -36,13 +37,23 @@
             <horizontal>
               <resolution>1</resolution>
+              <!--
               <samples>1875</samples>
               <min_angle>-3.1415926535897931</min_angle>
               <max_angle>3.1415926535897931</max_angle>
+              -->
+              <samples>600</samples>
+              <min_angle>${-PI}</min_angle>
+              <max_angle>${PI}</max_angle>
             </horizontal>
             <vertical>
               <resolution>1</resolution>
+              <!--
               <samples>16</samples>
               <min_angle>-0.26179938779</min_angle>
               <max_angle>0.26179938779</max_angle>
+              -->
+              <samples>9</samples>
+              <min_angle>${-PI/12}</min_angle>
+              <max_angle>${PI/180}</max_angle>
             </vertical>
           </scan>
