Commit message: apply format

File: orange_description/xacro/sensors/mid360.xacro (robot description, xacro)
@@ -8,8 +8,8 @@
   <xacro:property name="noise_mean" value="0.0"/>
   <xacro:property name="noise_stddev" value="0.01"/>
-  <xacro:property name="mass" value="0.4" />
-  <xacro:property name="length" value="0.1" />
-  <xacro:property name="width" value="0.06" />
-  <xacro:property name="height" value="0.06" />
+  <xacro:property name="mass" value="0.4"/>
+  <xacro:property name="length" value="0.1"/>
+  <xacro:property name="width" value="0.06"/>
+  <xacro:property name="height" value="0.06"/>
   <xacro:macro name="box_inertia" params="m w h d">
     <inertial>
@@ -20,12 +20,12 @@
   </xacro:macro>
   <xacro:macro name="mid360" params="name:='' parent:= 'base_link' topic:='mid360' *origin ">
-<link name="${name}">
-<xacro:box_inertia m="${length}" w="${width}" d="${length}" h="${height}"/>
-  <visual>
+    <link name="${name}">
+      <xacro:box_inertia m="${length}" w="${width}" d="${length}" h="${height}"/>
+      <visual>
         <geometry>
-            <box size="${length} ${width} ${height}"/>
+          <box size="${length} ${width} ${height}"/>
         </geometry>
-  </visual>
-</link>
+      </visual>
+    </link>
     <joint name="${name}_joint" type="fixed">
       <parent link="${parent}"/>
@@ -40,35 +40,35 @@
         <!-- This ray plgin is only for visualization. -->
         <plugin name="${name}_plugin" filename="libros2_livox.so">
-			<ray>
-			  <scan>
-				<horizontal>
-				<samples>100</samples>
-				<resolution>1</resolution>
-				<min_angle>${0}</min_angle>
-				<max_angle>${2*M_PI}</max_angle>
-				</horizontal>
-				<vertical>
-				<samples>360</samples>
-				<resolution>1</resolution>
-				<min_angle>${-7.22/180*M_PI}</min_angle>
-				<max_angle>${55.22/180*M_PI}</max_angle>
-				</vertical>
-			  </scan>
-			  <range>
-				<min>${laser_min_range}</min>
-				<max>${laser_max_range}</max>
-				<resolution>${resolution}</resolution>
-			  </range>
-			  <noise>
-				<type>gaussian</type>
-				<mean>${noise_mean}</mean>
-				<stddev>${noise_stddev}</stddev>
-			  </noise>
-			</ray>
+          <ray>
+            <scan>
+              <horizontal>
+                <samples>100</samples>
+                <resolution>1</resolution>
+                <min_angle>${0}</min_angle>
+                <max_angle>${2*M_PI}</max_angle>
+              </horizontal>
+              <vertical>
+                <samples>360</samples>
+                <resolution>1</resolution>
+                <min_angle>${-7.22/180*M_PI}</min_angle>
+                <max_angle>${55.22/180*M_PI}</max_angle>
+              </vertical>
+            </scan>
+            <range>
+              <min>${laser_min_range}</min>
+              <max>${laser_max_range}</max>
+              <resolution>${resolution}</resolution>
+            </range>
+            <noise>
+              <type>gaussian</type>
+              <mean>${noise_mean}</mean>
+              <stddev>${noise_stddev}</stddev>
+            </noise>
+          </ray>
           <visualize>false</visualize>
-		  <samples>${samples}</samples>
-		  <downsample>1</downsample>
-		  <csv_file_name>$(find ros2_livox_simulation)/scan_mode/mid360.csv</csv_file_name>
-		  <topic>${topic}</topic>
+          <samples>${samples}</samples>
+          <downsample>1</downsample>
+          <csv_file_name>$(find ros2_livox_simulation)/scan_mode/mid360.csv</csv_file_name>
+          <topic>${topic}</topic>
         </plugin>
       </sensor>
