Commit message: apply format

File: orange_description/xacro/orange_robot.xacro (robot description, xacro)
@@ -1,89 +1,85 @@
 <?xml version="1.0"?>
-<robot name="orange_robot" xmlns:xacro="http://www.ros.org/wiki/xacro">
+<robot xmlns:xacro="http://www.ros.org/wiki/xacro" name="orange_robot">
   <!--import gazebo reference-->
-  <xacro:include filename="$(find orange_description)/xacro/orange_robot.gazebo" />
+  <xacro:include filename="$(find orange_description)/xacro/orange_robot.gazebo"/>
   <!--import 2D LiDAR model-->
-  <xacro:include filename="$(find orange_description)/xacro/sensors/hokuyo.xacro" />
-  <xacro:sensor_hokuyo name="hokuyo" parent="base_link"
-    min_angle="-1.22" max_angle="1.22" samples="720">
-    <origin xyz="0.1075 0.0 0.1085" rpy="0.0 0.0 0.0" />
+  <xacro:include filename="$(find orange_description)/xacro/sensors/hokuyo.xacro"/>
+  <xacro:sensor_hokuyo name="hokuyo" parent="base_link" min_angle="-1.22" max_angle="1.22" samples="720">
+    <origin xyz="0.1075 0.0 0.1085" rpy="0.0 0.0 0.0"/>
   </xacro:sensor_hokuyo>
   <!--import 3D LiDAR model-->
-  <xacro:include filename="$(find orange_description)/xacro/sensors/velodyne.xacro" />
-  <xacro:sensor_velodyne name="velodyne" parent="base_link"
-    min_angle="-2.35619" max_angle="2.35619" samples="720">
-    <origin xyz="-0.0185 0.0 0.8985" rpy="0.0 0.0 0.0" />
+  <xacro:include filename="$(find orange_description)/xacro/sensors/velodyne.xacro"/>
+  <xacro:sensor_velodyne name="velodyne" parent="base_link" min_angle="-2.35619" max_angle="2.35619" samples="720">
+    <origin xyz="-0.0185 0.0 0.8985" rpy="0.0 0.0 0.0"/>
   </xacro:sensor_velodyne>
   <!--import imu model-->
-  <xacro:include filename="$(find orange_description)/xacro/sensors/imu.xacro" />
+  <xacro:include filename="$(find orange_description)/xacro/sensors/imu.xacro"/>
   <xacro:sensor_imu name="imu" parent="base_link" size="0.05 0.05 0.05">
-    <origin xyz="-0.253 0.0 0.068" rpy="0.0 0.0 0.0" />
+    <origin xyz="-0.253 0.0 0.068" rpy="0.0 0.0 0.0"/>
   </xacro:sensor_imu>
   <!--base footprint-->
-  <link name="base_footprint" />
+  <link name="base_footprint"/>
   <!--base link-->
   <joint name="base_joint" type="fixed">
-    <parent link="base_footprint" />
-    <child link="base_link" />
-    <origin xyz="0.0 0.0 0.1015" rpy="0 0 0" />
+    <parent link="base_footprint"/>
+    <child link="base_link"/>
+    <origin xyz="0.0 0.0 0.1015" rpy="0 0 0"/>
   </joint>
   <link name="base_link">
     <visual>
-      <origin xyz="0.0775 0.25275 0.6425" rpy="0.0 0.0 0.0" />
+      <origin xyz="0.0775 0.25275 0.6425" rpy="0.0 0.0 0.0"/>
       <geometry>
-        <mesh filename="file://$(find orange_description)/meshes/chassis.dae" />
+        <mesh filename="file://$(find orange_description)/meshes/chassis.dae"/>
       </geometry>
     </visual>
     <collision>
-      <origin xyz="-0.1995 0.0 0.341" rpy="0.0 0.0 0.0" />
+      <origin xyz="-0.1995 0.0 0.341" rpy="0.0 0.0 0.0"/>
       <geometry>
-        <box size="0.549 0.5055 0.603" />
+        <box size="0.549 0.5055 0.603"/>
       </geometry>
     </collision>
     <inertial>
-      <mass value="27.1" />
-      <origin xyz="-0.1995 0.0 0.19" rpy="0.0 0.0 0.0" />
-      <inertia ixx="0.78032248125" ixy="0.0" ixz="0.0" iyy="0.883913925" iyz="0.0"
-        izz="1.25773640625" />
+      <mass value="27.1"/>
+      <origin xyz="-0.1995 0.0 0.19" rpy="0.0 0.0 0.0"/>
+      <inertia ixx="0.78032248125" ixy="0.0" ixz="0.0" iyy="0.883913925" iyz="0.0" izz="1.25773640625"/>
     </inertial>
   </link>
   <!--caster-->
   <joint name="left_caster_hinge" type="fixed">
-    <origin xyz="0.0 0.0 0.0" rpy="0.0 0.0 0.0" />
-    <child link="left_caster_link" />
-    <parent link="base_link" />
+    <origin xyz="0.0 0.0 0.0" rpy="0.0 0.0 0.0"/>
+    <child link="left_caster_link"/>
+    <parent link="base_link"/>
   </joint>
   <joint name="right_caster_hinge" type="fixed">
-    <origin xyz="0.0 0.0 0.0" rpy="0.0 0.0 0.0" />
-    <child link="right_caster_link" />
-    <parent link="base_link" />
+    <origin xyz="0.0 0.0 0.0" rpy="0.0 0.0 0.0"/>
+    <child link="right_caster_link"/>
+    <parent link="base_link"/>
   </joint>
   <link name="left_caster_link">
     <visual>
-      <origin xyz="-0.4815 0.145 -0.039" rpy="0.0 0.0 0.0" />
+      <origin xyz="-0.4815 0.145 -0.039" rpy="0.0 0.0 0.0"/>
       <geometry>
-        <mesh filename="file://$(find orange_description)/meshes/left_caster.dae" />
+        <mesh filename="file://$(find orange_description)/meshes/left_caster.dae"/>
       </geometry>
     </visual>
     <collision>
-      <origin xyz="-0.4815 0.145 -0.039" rpy="0.0 1.57079632679 1.57079632679" />
+      <origin xyz="-0.4815 0.145 -0.039" rpy="0.0 1.57079632679 1.57079632679"/>
       <geometry>
-        <sphere radius="0.0625" />
+        <sphere radius="0.0625"/>
       </geometry>
     </collision>
   </link>
-  <link
-    name="right_caster_link">
+  <link name="right_caster_link">
     <visual>
-      <origin xyz="-0.4815 -0.145 -0.039" rpy="0.0 0.0 0.0" />
+      <origin xyz="-0.4815 -0.145 -0.039" rpy="0.0 0.0 0.0"/>
       <geometry>
-        <mesh filename="file://$(find orange_description)/meshes/right_caster.dae" />
-        <sphere radius="0.0625" />
+        <mesh filename="file://$(find orange_description)/meshes/right_caster.dae"/>
+        <sphere radius="0.0625"/>
       </geometry>
     </visual>
     <collision>
-      <origin xyz="-0.4815 -0.145 -0.039" rpy="0.0 1.57079632679 1.57079632679" />
+      <origin xyz="-0.4815 -0.145 -0.039" rpy="0.0 1.57079632679 1.57079632679"/>
       <geometry>
-        <sphere radius="0.0625" />
+        <sphere radius="0.0625"/>
       </geometry>
     </collision>
@@ -91,55 +87,53 @@
   <!--front wheels-->
   <joint type="revolute" name="left_wheel_hinge">
-    <origin xyz="0.0 0.2834 0.0" rpy="0.0 0.0 0.0" />
+    <origin xyz="0.0 0.2834 0.0" rpy="0.0 0.0 0.0"/>
     <child link="left_wheel">left_wheel</child>
     <parent link="base_link">base_link</parent>
-    <axis xyz="0 1 0" />
-    <limit effort="100" velocity="100.0" lower="-5000" upper="5000" />
+    <axis xyz="0 1 0"/>
+    <limit effort="100" velocity="100.0" lower="-5000" upper="5000"/>
   </joint>
   <joint type="revolute" name="right_wheel_hinge">
-    <origin xyz="0.0 -0.2834 0.0" rpy="0.0 0.0 0.0" />
+    <origin xyz="0.0 -0.2834 0.0" rpy="0.0 0.0 0.0"/>
     <child link="right_wheel">right_wheel</child>
     <parent link="base_link">base_link</parent>
-    <axis xyz="0 1 0" />
-    <limit effort="100" velocity="100.0" lower="-5000" upper="5000" />
+    <axis xyz="0 1 0"/>
+    <limit effort="100" velocity="100.0" lower="-5000" upper="5000"/>
   </joint>
   <link name="left_wheel">
     <visual name="visual">
-      <origin xyz="0.0 0.0 0.0" rpy="0.0 0.0 0.0" />
+      <origin xyz="0.0 0.0 0.0" rpy="0.0 0.0 0.0"/>
       <geometry>
-        <mesh filename="file://$(find orange_description)/meshes/front_wheel.dae" />
+        <mesh filename="file://$(find orange_description)/meshes/front_wheel.dae"/>
       </geometry>
     </visual>
     <collision name="collision">
-      <origin xyz="0.0 0.0 0.0" rpy="0.0 1.57079632679 1.57079632679" />
+      <origin xyz="0.0 0.0 0.0" rpy="0.0 1.57079632679 1.57079632679"/>
       <geometry>
-        <cylinder length="0.047" radius="0.1015" />
+        <cylinder length="0.047" radius="0.1015"/>
       </geometry>
     </collision>
     <inertial>
-      <mass value="3.4" />
-      <origin xyz="0.0 0.0 0.0" rpy="0.0 1.57079632679 1.57079632679" />
-      <inertia ixx="0.00938279583" ixy="0.0" ixz="0.0" iyy="0.00938279583" iyz="0.0"
-        izz="0.017513825" />
+      <mass value="3.4"/>
+      <origin xyz="0.0 0.0 0.0" rpy="0.0 1.57079632679 1.57079632679"/>
+      <inertia ixx="0.00938279583" ixy="0.0" ixz="0.0" iyy="0.00938279583" iyz="0.0" izz="0.017513825"/>
     </inertial>
   </link>
   <link name="right_wheel">
     <visual name="visual">
-      <origin xyz="0.0 0.0 0.0" rpy="0.0 0.0 0.0" />
+      <origin xyz="0.0 0.0 0.0" rpy="0.0 0.0 0.0"/>
       <geometry>
-        <mesh filename="file://$(find orange_description)/meshes/front_wheel.dae" />
+        <mesh filename="file://$(find orange_description)/meshes/front_wheel.dae"/>
       </geometry>
     </visual>
     <collision name="collision">
-      <origin xyz="0.0 0.0 0.0" rpy="0.0 1.57079632679 1.57079632679" />
+      <origin xyz="0.0 0.0 0.0" rpy="0.0 1.57079632679 1.57079632679"/>
       <geometry>
-        <cylinder length="0.047" radius="0.1015" />
+        <cylinder length="0.047" radius="0.1015"/>
       </geometry>
     </collision>
     <inertial>
-      <mass value="3.4" />
-      <origin xyz="0.0 0.0 0.0" rpy="0.0 1.57079632679 1.57079632679" />
-      <inertia ixx="0.00938279583" ixy="0.0" ixz="0.0" iyy="0.00938279583" iyz="0.0"
-        izz="0.017513825" />
+      <mass value="3.4"/>
+      <origin xyz="0.0 0.0 0.0" rpy="0.0 1.57079632679 1.57079632679"/>
+      <inertia ixx="0.00938279583" ixy="0.0" ixz="0.0" iyy="0.00938279583" iyz="0.0" izz="0.017513825"/>
     </inertial>
   </link>

File: orange_description/xacro/sensors/hokuyo.xacro (robot description, xacro)
@@ -1,30 +1,28 @@
 <?xml version="1.0"?>
-<robot name="sensor_hokuyo" xmlns:xacro="http://ros.org/wiki/xacro"
-  xmlns:controller="http://playerstage.sourceforge.net/gazebo/xmlschema/#controller"
-  xmlns:interface="http://playerstage.sourceforge.net/gazebo/xmlschema/#interface">
+<robot xmlns:xacro="http://ros.org/wiki/xacro" xmlns:controller="http://playerstage.sourceforge.net/gazebo/xmlschema/#controller" xmlns:interface="http://playerstage.sourceforge.net/gazebo/xmlschema/#interface" name="sensor_hokuyo">
   <xacro:macro name="sensor_hokuyo" params="name parent *origin min_angle max_angle samples">
     <joint name="${name}_joint" type="fixed">
-      <xacro:insert_block name="origin" />
-      <axis xyz="0 1 0" />
-      <parent link="${parent}" />
-      <child link="${name}_link" />
+      <xacro:insert_block name="origin"/>
+      <axis xyz="0 1 0"/>
+      <parent link="${parent}"/>
+      <child link="${name}_link"/>
     </joint>
     <link name="${name}_link">
       <visual>
-        <origin xyz="0 0 0" rpy="0 0 0" />
+        <origin xyz="0 0 0" rpy="0 0 0"/>
         <geometry>
-          <mesh filename="file://$(find orange_description)/meshes/hokuyo.dae" />
+          <mesh filename="file://$(find orange_description)/meshes/hokuyo.dae"/>
         </geometry>
       </visual>
       <collision>
-        <origin xyz="0 0 0" rpy="0 0 0" />
+        <origin xyz="0 0 0" rpy="0 0 0"/>
         <geometry>
-          <box size="0.1 0.1 0.1" />
+          <box size="0.1 0.1 0.1"/>
         </geometry>
       </collision>
       <inertial>
-        <mass value="0.0001" />
-        <origin xyz="0 0 0" rpy="0 0 0" />
-        <inertia ixx="0.0001" ixy="0" ixz="0" iyy="0.0001" iyz="0" izz="0.0001" />
+        <mass value="0.0001"/>
+        <origin xyz="0 0 0" rpy="0 0 0"/>
+        <inertia ixx="0.0001" ixy="0" ixz="0" iyy="0.0001" iyz="0" izz="0.0001"/>
       </inertial>
     </link>

File: orange_description/xacro/sensors/imu.xacro (robot description, xacro)
@@ -1,30 +1,28 @@
 <?xml version="1.0"?>
-<robot name="sensor_imu" xmlns:xacro="http://ros.org/wiki/xacro"
-  xmlns:controller="http://playerstage.sourceforge.net/gazebo/xmlschema/#controller"
-  xmlns:interface="http://playerstage.sourceforge.net/gazebo/xmlschema/#interface">
+<robot xmlns:xacro="http://ros.org/wiki/xacro" xmlns:controller="http://playerstage.sourceforge.net/gazebo/xmlschema/#controller" xmlns:interface="http://playerstage.sourceforge.net/gazebo/xmlschema/#interface" name="sensor_imu">
   <xacro:macro name="sensor_imu" params="name parent *origin size">
     <joint name="${name}_joint" type="fixed">
-      <xacro:insert_block name="origin" />
-      <axis xyz="1 0 0" />
-      <parent link="${parent}" />
-      <child link="${name}_link" />
+      <xacro:insert_block name="origin"/>
+      <axis xyz="1 0 0"/>
+      <parent link="${parent}"/>
+      <child link="${name}_link"/>
     </joint>
     <link name="${name}_link">
       <visual>
-        <origin rpy="0 0 0" xyz="0 0 0" />
+        <origin rpy="0 0 0" xyz="0 0 0"/>
         <geometry>
-          <box size="${size}" />
+          <box size="${size}"/>
         </geometry>
       </visual>
       <collision>
-        <origin rpy="0 0 0" xyz="0 0 0" />
+        <origin rpy="0 0 0" xyz="0 0 0"/>
         <geometry>
-          <box size="${size}" />
+          <box size="${size}"/>
         </geometry>
       </collision>
       <inertial>
-        <mass value="0.001" />
-        <origin rpy="0 0 0" xyz="0 0 0" />
-        <inertia ixx="0.0001" ixy="0" ixz="0" iyy="0.000001" iyz="0" izz="0.0001" />
+        <mass value="0.001"/>
+        <origin rpy="0 0 0" xyz="0 0 0"/>
+        <inertia ixx="0.0001" ixy="0" ixz="0" iyy="0.000001" iyz="0" izz="0.0001"/>
       </inertial>
     </link>

File: orange_description/xacro/sensors/velodyne.xacro (robot description, xacro)
@@ -1,30 +1,28 @@
 <?xml version="1.0"?>
-<robot name="sensor_velodyne" xmlns:xacro="http://ros.org/wiki/xacro"
-  xmlns:controller="http://playerstage.sourceforge.net/gazebo/xmlschema/#controller"
-  xmlns:interface="http://playerstage.sourceforge.net/gazebo/xmlschema/#interface">
+<robot xmlns:xacro="http://ros.org/wiki/xacro" xmlns:controller="http://playerstage.sourceforge.net/gazebo/xmlschema/#controller" xmlns:interface="http://playerstage.sourceforge.net/gazebo/xmlschema/#interface" name="sensor_velodyne">
   <xacro:macro name="sensor_velodyne" params="name parent *origin min_angle max_angle samples">
     <joint name="${name}_joint" type="fixed">
-      <xacro:insert_block name="origin" />
-      <axis xyz="0 1 0" />
-      <parent link="${parent}" />
-      <child link="${name}_link" />
+      <xacro:insert_block name="origin"/>
+      <axis xyz="0 1 0"/>
+      <parent link="${parent}"/>
+      <child link="${name}_link"/>
     </joint>
     <link name="${name}_link">
       <visual>
-        <origin xyz="0 0 0" rpy="0 0 0" />
+        <origin xyz="0 0 0" rpy="0 0 0"/>
         <geometry>
-          <mesh filename="file://$(find orange_description)/meshes/velodyne.dae" />
+          <mesh filename="file://$(find orange_description)/meshes/velodyne.dae"/>
         </geometry>
       </visual>
       <collision>
-        <origin xyz="0 0 0" rpy="0 0 0" />
+        <origin xyz="0 0 0" rpy="0 0 0"/>
         <geometry>
-          <box size="0.1 0.1 0.1" />
+          <box size="0.1 0.1 0.1"/>
         </geometry>
       </collision>
       <inertial>
-        <mass value="0.0001" />
-        <origin xyz="0 0 0" rpy="0 0 0" />
-        <inertia ixx="0.0001" ixy="0" ixz="0" iyy="0.0001" iyz="0" izz="0.0001" />
+        <mass value="0.0001"/>
+        <origin xyz="0 0 0" rpy="0 0 0"/>
+        <inertia ixx="0.0001" ixy="0" ixz="0" iyy="0.0001" iyz="0" izz="0.0001"/>
       </inertial>
     </link>

Commit message: feature livox_slam

File: orange_description/xacro/orange_robot.xacro (robot description, xacro)
@@ -9,8 +9,8 @@
   </xacro:sensor_hokuyo>
   <!--import 3D LiDAR model-->
-  <xacro:include filename="$(find orange_description)/xacro/sensors/velodyne.xacro"/>
-  <xacro:sensor_velodyne name="velodyne" parent="base_link" min_angle="-2.35619" max_angle="2.35619" samples="720">
-    <origin xyz="-0.0185 0.0 0.8985" rpy="0.0 0.0 0.0"/>
-  </xacro:sensor_velodyne>
+  <xacro:include filename="$(find orange_description)/xacro/sensors/livox.xacro"/>
+  <xacro:sensor_livox name="livox_frame" parent="base_link" min_angle="-2.35619" max_angle="2.35619" samples="720">
+    <origin xyz="-0.0185 0.0 0.8985" rpy="${pi} 0.0 0.0"/>
+  </xacro:sensor_livox>
   <!--import imu model-->
   <xacro:include filename="$(find orange_description)/xacro/sensors/imu.xacro"/>

Commit message: feature simulation

File: orange_description/xacro/orange_robot.xacro (robot description, xacro)
@@ -9,8 +9,14 @@
   </xacro:sensor_hokuyo>
   <!--import 3D LiDAR model-->
+  <!--bringup-->
   <xacro:include filename="$(find orange_description)/xacro/sensors/livox.xacro"/>
   <xacro:sensor_livox name="livox_frame" parent="base_link" min_angle="-2.35619" max_angle="2.35619" samples="720">
     <origin xyz="-0.0185 0.0 0.8985" rpy="${pi} 0.0 0.0"/>
   </xacro:sensor_livox>
+  <!--simulation-->
+  <!--<xacro:include filename="$(find ros2_livox_simulation)/urdf/mid360.xacro"/>
+  <xacro:mid360 name="livox" parent="base_link" topic="mid360">
+    <origin xyz="-0.0185 0.0 0.8985" rpy="${pi} 0.0 0.0"/>
+  </xacro:mid360>-->
   <!--import imu model-->
   <xacro:include filename="$(find orange_description)/xacro/sensors/imu.xacro"/>

Commit message: fix/ground_segmentation

File: orange_description/xacro/orange_robot.xacro (robot description, xacro)
@@ -12,5 +12,6 @@
   <xacro:include filename="$(find orange_description)/xacro/sensors/livox.xacro"/>
   <xacro:sensor_livox name="livox_frame" parent="base_link" min_angle="-2.35619" max_angle="2.35619" samples="720">
-    <origin xyz="-0.0185 0.0 0.8985" rpy="${pi} 0.0 0.0"/>
+    <origin xyz="0.0 0.0 0.0" rpy="0.0 0.0 0.0"/>
+    <!-- <origin xyz="-0.0185 0.0 0.8985" rpy="${pi} 0.0 0.0"/> -->
   </xacro:sensor_livox>
   <!--simulation-->

Commit message: xacro file adding tof senesor

File: orange_description/xacro/orange_robot.xacro (robot description, xacro)
@@ -8,4 +8,9 @@
     <origin xyz="0.1075 0.0 0.1085" rpy="0.0 0.0 0.0"/>
   </xacro:sensor_hokuyo>
+  <!-- ToFセンサー (VL53L5CX) の追加 -->
+  <xacro:include filename="$(find orange_description)/xacro/sensors/tof.xacro"/>
+  <xacro:sensor_vl53l5cx name="tof_sensor" parent="base_link">
+    <origin xyz="0.1075 0.025 0.1085" rpy="0.0 0.0 0.0"/> <!-- LiDARのすぐ横に配置 -->
+  </xacro:sensor_vl53l5cx>
   <!--import 3D LiDAR model-->
   <!--bringup-->
